File: c99.kicad_pcb (KiCad board)
At the start: 4 copper layers, 100 x 100 mm, 52 parts, among them J1 Reset, J3 Serial, J4 +5V, J5 Bus, SW1 Reset, SW2 Power, U1 TMS9995, U10 74LS259, U12 74LS74, U13 74LS112, U14 74LS138, U2 74LS612, U3 74LS14, U4 28C256, U5 AS6C4008-55PCN, U6 74LS688, U7 GAL22V10, U8 TMS9902, Y1 12MHz

Commit message: silkscreen fixups
Parts:
- added LOGO1: crankery, c99:crankery_small, F.Cu at (115.2, 29.6)
- added LOGO2: cortex, c99:cortex, F.Cu at (82.5, 121.9)
- added LOGO3: cortex, c99:eti, F.Cu at (122.3, 36.5)
- C1, C10, C11, C12, C13, C14, C15, C16, C2, C5, C6, C7, C8, C9: footprint Capacitor_THT:C_Disc_D4.3mm_W1.9mm_P5.00mm -> c99:C_Disc_D4.3mm_W1.9mm_P5.00mm
- C3, C4: footprint Capacitor_THT:CP_Radial_D5.0mm_P2.00mm -> c99:CP_Radial_D5.0mm_P2.00mm
- D2, D4, D5: footprint LED_THT:LED_D3.0mm -> c99:LED_D3.0mm
- D3: footprint Diode_THT:D_DO-41_SOD81_P7.62mm_Horizontal -> c99:D_DO-41_SOD81_P7.62mm_Horizontal
- H1, H2, H3, H4: footprint MountingHole:MountingHole_2.7mm_M2.5_DIN965_Pad -> c99:MountingHole_2.7mm_M2.5_DIN965_Pad
- J1: footprint Connector_JST:JST_PH_B2B-PH-K_1x02_P2.00mm_Vertical -> c99:JST_PH_B2B-PH-K_1x02_P2.00mm_Vertical
- J3: footprint Connector_PinSocket_2.54mm:PinSocket_1x06_P2.54mm_Horizontal -> c99:PinSocket_1x06_P2.54mm_Horizontal
- J4: footprint Connector_BarrelJack:BarrelJack_Horizontal -> c99:BarrelJack_Horizontal
- J5: footprint Connector_PinHeader_2.54mm:PinHeader_2x25_P2.54mm_Vertical -> c99:PinHeader_2x25_P2.54mm_Vertical
- JP1, JP2: footprint Connector_PinHeader_2.54mm:PinHeader_1x02_P2.54mm_Vertical -> c99:PinHeader_1x02_P2.54mm_Vertical
- R12, R13, R14, R15, R16, R17, R3: footprint Resistor_THT:R_Axial_DIN0204_L3.6mm_D1.6mm_P5.08mm_Horizontal -> c99:R_Axial_DIN0204_L3.6mm_D1.6mm_P5.08mm_Horizontal
- SW1: footprint Button_Switch_THT:SW_Tactile_SPST_Angled_PTS645Vx39-2LFS -> c99:SW_Tactile_SPST_Angled_PTS645Vx39-2LFS
- U1, U2: footprint Package_DIP:DIP-40_W15.24mm -> c99:DIP-40_W15.24mm
- U10, U13, U14: footprint Package_DIP:DIP-16_W7.62mm -> c99:DIP-16_W7.62mm
- U12, U3: footprint Package_DIP:DIP-14_W7.62mm -> c99:DIP-14_W7.62mm
- U4: footprint Package_DIP:DIP-28_W15.24mm -> c99:DIP-28_W15.24mm
- U5: footprint Package_DIP:DIP-32_W15.24mm -> c99:DIP-32_W15.24mm
- U6: footprint Package_DIP:DIP-20_W7.62mm -> c99:DIP-20_W7.62mm
- U7: footprint Package_DIP:DIP-24_W7.62mm -> c99:DIP-24_W7.62mm
- U8: footprint Package_DIP:DIP-18_W7.62mm -> c99:DIP-18_W7.62mm
- Y1: footprint Crystal:Crystal_HC49-U_Vertical -> c99:Crystal_HC49-U_Vertical
- moved C4 21.6 mm to (106.3, 27.4)
Other:
- board text added: "(1)"
- board text added: "(50)"
- board text added: "+5V"
- board text added: "AB0"
- board text added: "AB1"
- board text added: "AB10"
- board text added: "AB11"
- board text added: "AB2"
- board text added: "AB3"
- board text added: "AB4"
- board text added: "AB5"
- board text added: "AB6"
- board text added: "AB7"
- board text added: "AB8"
- board text added: "AB9"
- board text added: "CLKOUT"
- board text added: "CRUIN"
- board text added: "D0"
- board text added: "D1"
- board text added: "D2"
- board text added: "D3"
- board text added: "D4"
- board text added: "D5"
- board text added: "D6"
- board text added: "D7"
- board text added: "FLAG1"
- board text added: "FLAG2"
- board text added: "FLAG3"
- board text added: "FLAG4"
- board text added: "GND"
- board text added: "IAQ"
- board text added: "Mini^{2}"
- board text added: "Mini^{2}Cortex v1 2026-07-06"
- board text added: "RA12"
- board text added: "RA13"
- board text added: "RA14"
- board text added: "RA15"
- board text added: "READY"
- board text added: "Stuart Conner - design Dave Hamilton - layout"
- board text added: "USER"
- board text added: "WAIT"
- board text added: "~{CFSEL}"
- board text added: "~{CRUCLK}"
- board text added: "~{CSR}"
- board text added: "~{CSW}"
- board text added: "~{DBIN}"
- board text added: "~{HOLD}"
- board text added: "~{INT1}"
- board text added: "~{INT4}"
- board text added: "~{MENEN}"
- board text added: "~{NMI}"
- board text added: "~{PWE}"
- board text added: "~{RESET}"
